Commit message: added DJI F450 model to RotorS

File: rotors_description/urdf/iris.xacro (robot description, xacro)
@@ -3,27 +3,31 @@
   <!-- Properties -->
   <xacro:property name="namespace" value="$(arg namespace)" />
-  <xacro:property name="rotor_velocity_slowdown_sim" value="10" />
+  <xacro:property name="rotor_velocity_slowdown_sim" value="10" /> <!-- what is this??? -->
   <xacro:property name="use_mesh_file" value="true" />
-  <xacro:property name="mesh_file" value="package://rotors_description/meshes/iris.dae" />
-  <xacro:property name="mass" value="1.5" /> <!-- [kg] -->
-  <xacro:property name="body_width" value="0.47" /> <!-- [m] -->
-  <xacro:property name="body_height" value="0.11" /> <!-- [m] -->
-  <xacro:property name="mass_rotor" value="0.005" /> <!-- [kg] -->
-  <xacro:property name="arm_length_front_x" value="0.13" /> <!-- [m] -->
-  <xacro:property name="arm_length_back_x" value="0.13" /> <!-- [m] -->
-  <xacro:property name="arm_length_front_y" value="0.22" /> <!-- [m] -->
-  <xacro:property name="arm_length_back_y" value="0.2" /> <!-- [m] -->
-  <xacro:property name="rotor_offset_top" value="0.023" /> <!-- [m] -->
-  <xacro:property name="radius_rotor" value="0.1" /> <!-- [m] -->
-  <xacro:property name="motor_constant" value="8.54858e-06" /> <!-- [kg.m/s^2] -->
-  <xacro:property name="moment_constant" value="0.016" /> <!-- [m] -->
-  <xacro:property name="time_constant_up" value="0.0125" /> <!-- [s] -->
-  <xacro:property name="time_constant_down" value="0.025" /> <!-- [s] -->
+  <xacro:property name="mesh_file" value="package://rotors_description/meshes/Assemprt1.sldprt.STL" />
+  <xacro:property name="mass" value="0.985" /> <!-- [kg] -->
+  <xacro:property name="body_radius" value="0.355" /> <!-- [m] -->
+  <xacro:property name="body_length" value="0.213" /> <!-- [m] -->
+  <xacro:property name="mass_rotor" value="0.013" /> <!-- [kg] -->
+  <xacro:property name="arm_one_x" value="0.227856" /> <!-- [m] -->
+  <xacro:property name="arm_one_y" value="-0.003669881" /> <!-- [m]-->
+  <xacro:property name="arm_two_x" value="0.002071819" /> <!-- [m] -->
+  <xacro:property name="arm_two_y" value="0.222" /> <!-- [m]-->
+  <xacro:property name="arm_three_x" value="-0.223712362" /> <!-- [m] -->
+  <xacro:property name="arm_three_y" value="-0.003669881" /> <!-- [m]-->
+  <xacro:property name="arm_four_x" value="0.00224186" /> <!-- [m] -->
+  <xacro:property name="arm_four_y" value="-0.2295" /> <!-- [m]-->
+  <xacro:property name="rotor_offset_top" value="0.05921" /> <!-- [m] -->
+  <xacro:property name="radius_rotor" value="1" /> <!-- [m] -->
+  <xacro:property name="motor_constant" value="8.54858e-06" /> <!-- [kg.m/s^2] --> <!-- what is this??? -->
+  <xacro:property name="moment_constant" value="0.016" /> <!-- [m] --> <!-- what is this??? -->
+  <xacro:property name="time_constant_up" value="0.0125" /> <!-- [s] --> <!-- what is this??? -->
+  <xacro:property name="time_constant_down" value="0.025" /> <!-- [s] --> <!-- what is this??? -->
   <xacro:property name="max_rot_velocity" value="838" /> <!-- [rad/s] -->
   <xacro:property name="sin30" value="0.5" />
   <xacro:property name="cos30" value="0.866025403784" />
   <xacro:property name="sqrt2" value="1.4142135623730951" />
-  <xacro:property name="rotor_drag_coefficient" value="8.06428e-05" />
-  <xacro:property name="rolling_moment_coefficient" value="0.000001" />
+  <xacro:property name="rotor_drag_coefficient" value="8.06428e-05" /> <!-- what is this??? -->
+  <xacro:property name="rolling_moment_coefficient" value="0.000001" /> <!-- what is this??? -->
   <!-- Property Blocks -->
   <xacro:property name="body_inertia">
@@ -40,6 +44,6 @@
     robot_namespace="${namespace}"
     mass="${mass}"
-    body_width="${body_width}"
-    body_height="${body_height}"
+    body_radius="${body_radius}"
+    body_length="${body_length}"
     use_mesh_file="${use_mesh_file}"
     mesh_file="${mesh_file}"
@@ -64,7 +68,28 @@
     rolling_moment_coefficient="${rolling_moment_coefficient}"
     color="Blue"
-    use_own_mesh="false"
-    mesh="">
-    <origin xyz="${arm_length_front_x} -${arm_length_front_y} ${rotor_offset_top}" rpy="0 0 0" />
+    use_own_mesh="true"
+    mesh="package://rotors_description/meshes/prop1.sldprt.STL">
+    <origin xyz="${arm_one_x} ${arm_one_y} ${rotor_offset_top}" rpy="0 0 0" />
+    <xacro:insert_block name="rotor_inertia" />
+  </xacro:vertical_rotor>
+  <xacro:vertical_rotor
+    robot_namespace="${namespace}"
+    suffix="front left"
+    direction="cw"
+    motor_constant="${motor_constant}"
+    moment_constant="${moment_constant}"
+    parent="${namespace}/base_link"
+    mass_rotor="${mass_rotor}"
+    radius_rotor="${radius_rotor}"
+    time_constant_up="${time_constant_up}"
+    time_constant_down="${time_constant_down}"
+    max_rot_velocity="${max_rot_velocity}"
+    motor_number="1"
+    rotor_drag_coefficient="${rotor_drag_coefficient}"
+    rolling_moment_coefficient="${rolling_moment_coefficient}"
+    color="Red"
+    use_own_mesh="true"
+    mesh="package://rotors_description/meshes/prop1.sldprt.STL">
+    <origin xyz="${arm_two_x} ${arm_two_y} ${rotor_offset_top}" rpy="0 0 0" />
     <xacro:insert_block name="rotor_inertia" />
   </xacro:vertical_rotor>
@@ -81,35 +106,16 @@
     time_constant_down="${time_constant_down}"
     max_rot_velocity="${max_rot_velocity}"
-    motor_number="1"
-    rotor_drag_coefficient="${rotor_drag_coefficient}"
-    rolling_moment_coefficient="${rolling_moment_coefficient}"
-    color="Red"
-    use_own_mesh="false"
-    mesh="">
-    <origin xyz="-${arm_length_back_x} ${arm_length_back_y} ${rotor_offset_top}" rpy="0 0 0" />
-    <xacro:insert_block name="rotor_inertia" />
-  </xacro:vertical_rotor>
-  <xacro:vertical_rotor robot_namespace="${namespace}"
-    suffix="front_left"
-    direction="cw"
-    motor_constant="${motor_constant}"
-    moment_constant="${moment_constant}"
-    parent="${namespace}/base_link"
-    mass_rotor="${mass_rotor}"
-    radius_rotor="${radius_rotor}"
-    time_constant_up="${time_constant_up}"
-    time_constant_down="${time_constant_down}"
-    max_rot_velocity="${max_rot_velocity}"
     motor_number="2"
     rotor_drag_coefficient="${rotor_drag_coefficient}"
     rolling_moment_coefficient="${rolling_moment_coefficient}"
     color="Blue"
-    use_own_mesh="false"
-    mesh="">
-    <origin xyz="${arm_length_front_x} ${arm_length_front_y} ${rotor_offset_top}" rpy="0 0 0" />
+    use_own_mesh="true"
+    mesh="package://rotors_description/meshes/prop1.sldprt.STL">
+    <origin xyz="${arm_three_x} ${arm_three_y} ${rotor_offset_top}" rpy="0 0 0" />
     <xacro:insert_block name="rotor_inertia" />
   </xacro:vertical_rotor>
-  <xacro:vertical_rotor robot_namespace="${namespace}"
-    suffix="back_right"
+  <xacro:vertical_rotor
+    robot_namespace="${namespace}"
+    suffix="front_right"
     direction="cw"
     motor_constant="${motor_constant}"
@@ -125,8 +131,26 @@
     rolling_moment_coefficient="${rolling_moment_coefficient}"
     color="Red"
-    use_own_mesh="false"
-    mesh="">
-    <origin xyz="-${arm_length_back_x} -${arm_length_back_y} ${rotor_offset_top}" rpy="0 0 0" />
+    use_own_mesh="true"
+    mesh="package://rotors_description/meshes/prop1.sldprt.STL">
+    <origin xyz="${arm_four_x} ${arm_four_y} ${rotor_offset_top}" rpy="0 0 0" />
     <xacro:insert_block name="rotor_inertia" />
   </xacro:vertical_rotor>
+  <!--Mount a Camera-->
+  <xacro:camera_macro
+    namespace="${namespace}"
+    parent_link="${namespace}/base_link"
+    camera_suffix="nadir"
+    frame_rate="20.0"
+    horizontal_fov="2"
+    image_width="752"
+    image_height="480"
+    image_format="L8"
+    min_distance="0.02"
+    max_distance="50"
+    noise_mean="0.0"
+    noise_stddev="0.007"
+    enable_visual="true">
+      <box size="0.05 0.05 0.02" />
+      <origin xyz="${arm_one_x/4} ${arm_two_y/4} ${-arm_one_x/4}" rpy="0 ${pi/2} 0" />
+  </xacro:camera_macro>
 </robot>
