Commit message: DJI model updates

File: rotors_description/urdf/DJI_base.xacro (robot description, xacro)
@@ -10,31 +10,4 @@
     <xacro:default_mavlink_interface namespace="${namespace}" imu_sub_topic="imu" rotor_count="4" />
   </xacro:if>
-<!--Mount a Camera-->
-  <xacro:camera_macro
-    namespace="${namespace}"
-    parent_link="${namespace}/base_link"
-    camera_suffix="nadir"
-    frame_rate="20.0"
-    horizontal_fov="2"
-    image_width="752"
-    image_height="480"
-    image_format="R8G8B8"
-    min_distance="0.02"
-    max_distance="50"
-    noise_mean="0.0"
-    noise_stddev="0.007"
-    enable_visual="true">
-    <box size="0.023 0.0288 0.02955" />
-    <origin xyz=".04459 .03925 -.05168" rpy="0 1.5708 0.785398" />
-  </xacro:camera_macro>
-<!--Mount Stereo Camera -->
-  <xacro:vi_sensor_macro
-      namespace="${namespace}/vi_sensor"
-      parent_link="${namespace}/base_link"
-      enable_cameras="true"
-      enable_depth="true"
-      enable_ground_truth="true">
-    <origin xyz=".06459 .05925 -.10168" rpy="0.0 0.0 ${pi/4}" />
-  </xacro:vi_sensor_macro>
   <!-- Mount an ADIS16448 IMU. -->
   <xacro:default_imu namespace="${namespace}" parent_link="${namespace}/base_link" />
