Commit message: matrice and camera updates

File: rotors_description/urdf/component_snippets_MAIN_WITH_CAM_WEIGHTS.xacro (robot description, xacro)
@@ -683,5 +683,5 @@
       </visual>
       <inertial>
-        <mass value="0.001" />
+        <mass value="0.13" />
         <origin xyz="0 0 0" rpy="0 0 0" />
         <inertia ixx="1e-6" ixy="0" ixz="0" iyy="1e-6" iyz="0" izz="1e-6" />
@@ -896,5 +896,5 @@
       </visual>
       <inertial>
-        <mass value="0.001" />
+        <mass value="0.159" />
         <origin xyz="0 0 0" rpy="0 0 0" />
         <inertia ixx="1e-6" ixy="0" ixz="0" iyy="1e-6" iyz="0" izz="1e-6" />
